File: daughter/steering-wheel-daughter-boards.kicad_pcb (KiCad board)
At the start: 2 copper layers, 43.8 x 20 mm, 23 parts, among them J1 Conn_01x02_Socket, J2 Conn_01x06_Socket, SW3 SW_SPDT, SW4 SW_SPDT, U3 74HC14

Commit message: Fix DRC errors
Parts:
- moved H2 0.75 mm to (156.0, 76.2)
- moved J2 0.33 mm to (160.3, 72.5)
- moved R9 0.10 mm to (151.7, 77.2)
Routing:
- net BTN2: track 14.3 -> 13.0 mm, vias 0 -> 1
Changed lines of the file:
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@@
 	(footprint "Connector_JST:JST_EH_S6B-EH_1x06_P2.50mm_Horizontal"
 		(layer "F.Cu")
-		(at 159.9675 72.5 -90)
+		(at 160.3 72.5 -90)
 		(descr "JST EH series connector, S6B-EH (http://www.jst-mfg.com/product/pdf/eng/eEH.pdf), generated with kicad-footprint-generator")
 		(tags "connector JST EH horizontal")
@@
 		(tags "connector JST EH horizontal")
 		(property "Reference" "J1"
-			(at 1.25 -7.9 90)
+			(at 1.8 3.8675 90)
 			(layer "F.SilkS")
 			(effects
@@
 	(footprint "MountingHole:MountingHole_2.2mm_M2_ISO7380_Pad"
 		(layer "F.Cu")
-		(at 156 77)
+		(at 156 76.25)
 		(descr "Mounting Hole 2.2mm, M2, generated by kicad-footprint-generator mountinghole.py")
 		(tags "mountinghole M2 ISO7380")
@@
 	(footprint "Resistor_SMD:R_1206_3216Metric"
 		(layer "F.Cu")
-		(at 151.7125 77.25 180)
+		(at 151.7125 77.15 180)
 		(descr "Resistor SMD 1206 (3216 Metric), square (rectangular) end terminal, IPC-7351 nominal, (Body size source: IPC-SM-782 page 72, https://www.pcb-3d.com/wordpress/wp-content/uploads/ipc-sm-782a_amendment_1_and_2.pdf), generated with kicad-footprint-generator")
 		(tags "resistor")
@@
 	)
 	(segment
-		(start 158.8685 73.901)
-		(end 159.9675 75)
+		(start 153.52566 75.7)
+		(end 155.32466 73.901)
 		(width 0.2)
 		(layer "F.Cu")
@@
 	)
 	(segment
-		(start 136.7125 77.25)
-		(end 138.5375 77.25)
+		(start 149.4 75.7)
+		(end 153.52566 75.7)
 		(width 0.2)
 		(layer "F.Cu")
@@
 	)
 	(segment
-		(start 140.599 75.1885)
-		(end 140.599 73.88984)
+		(start 136.7125 77.25)
+		(end 138.5375 77.25)
 		(width 0.2)
 		(layer "F.Cu")
@@
 	)
 	(segment
-		(start 146.67934 75.926)
-		(end 150.79766 75.926)
+		(start 155.32466 73.901)
+		(end 158.8685 73.901)
 		(width 0.2)
 		(layer "F.Cu")
@@
 	)
 	(segment
-		(start 140.91484 73.574)
-		(end 146.04766 73.574)
+		(start 140.599 75.1885)
+		(end 140.599 73.88984)
 		(width 0.2)
 		(layer "F.Cu")
@@
 	)
 	(segment
-		(start 140.599 73.88984)
-		(end 140.91484 73.574)
+		(start 138.5375 77.25)
+		(end 140.599 75.1885)
 		(width 0.2)
 		(layer "F.Cu")
@@
 	)
 	(segment
-		(start 151.05066 75.673)
-		(end 153.55266 75.673)
+		(start 140.599 73.88984)
+		(end 140.91484 73.574)
 		(width 0.2)
 		(layer "F.Cu")
@@
 	)
 	(segment
-		(start 146.67934 74.20568)
-		(end 146.67934 75.926)
+		(start 140.91484 73.574)
+		(end 146.04766 73.574)
 		(width 0.2)
 		(layer "F.Cu")
@@
 	)
 	(segment
-		(start 138.5375 77.25)
-		(end 140.599 75.1885)
+		(start 146.67934 75.926)
+		(end 149.174 75.926)
 		(width 0.2)
 		(layer "F.Cu")
@@
 	)
 	(segment
-		(start 150.79766 75.926)
-		(end 151.05066 75.673)
+		(start 158.8685 73.901)
+		(end 159.9675 75)
 		(width 0.2)
 		(layer "F.Cu")
@@
 	)
 	(segment
-		(start 153.55266 75.673)
-		(end 155.32466 73.901)
+		(start 146.67934 74.20568)
+		(end 146.67934 75.926)
 		(width 0.2)
 		(layer "F.Cu")
@@
 	)
 	(segment
-		(start 155.32466 73.901)
-		(end 158.8685 73.901)
+		(start 149.174 75.926)
+		(end 149.4 75.7)
 		(width 0.2)
 		(layer "F.Cu")
@@
 	)
 	(segment
-		(start 157.052 74.302)
-		(end 155.49466 74.302)
+		(start 151.75 77.2)
+		(end 150.3 77.2)
 		(width 0.2)
 		(layer "F.Cu")
@@
 	)
 	(segment
-		(start 155.49466 74.302)
-		(end 153.72266 76.074)
-		(width 0.2)
-		(layer "F.Cu")
-		(net 7)
-	)
-	(segment
-		(start 151.25 76.25)
+		(start 150.3 77.2)
 		(end 150.25 77.25)
 		(width 0.2)
@@
 	)
 	(segment
-		(start 152.62734 76.074)
-		(end 152.45134 76.25)
+		(start 148.425 77.25)
+		(end 150.25 77.25)
 		(width 0.2)
 		(layer "F.Cu")
 		(net 7)
 	)
-	(segment
-		(start 159.9675 77.2175)
-		(end 157.052 74.302)
-		(width 0.2)
-		(layer "F.Cu")
+	(via
+		(at 151.75 77.2)
+		(size 0.6)
+		(drill 0.3)
+		(layers "F.Cu" "B.Cu")
 		(net 7)
 	)
 	(segment
-		(start 153.72266 76.074)
-		(end 152.62734 76.074)
+		(start 159.9675 77.5)
+		(end 158.7675 78.7)
 		(width 0.2)
-		(layer "F.Cu")
+		(layer "B.Cu")
 		(net 7)
 	)
 	(segment
-		(start 152.45134 76.25)
-		(end 151.25 76.25)
+		(start 153.25 78.7)
+		(end 151.75 77.2)
 		(width 0.2)
-		(layer "F.Cu")
+		(layer "B.Cu")
 		(net 7)
 	)
 	(segment
-		(start 148.425 77.25)
-		(end 150.25 77.25)
+		(start 158.7675 78.7)
+		(end 153.25 78.7)
 		(width 0.2)
-		(layer "F.Cu")
+		(layer "B.Cu")
 		(net 7)
 	)
